Commit message: nav2改为python编译，修复无法读取到文件的问题 修复simple_bot_description描述文件 降低卡尔曼滤波频率

File: Nodes/sam_bot_description/src/description/simple_bot.urdf (robot description, URDF)
Before this commit: robot simple_bot, 2 links, 1 joints
Joints:
- joint lidar_joint: origin xyz=0 -0.09 0.19 rpy=0 0 0 -> xyz=${-wheel_base/2} ${wheel_separation/2 - 0.09} ${-base_height/2 + wheel_radius + 0.19} rpy=0 0 0

Commit message: 更新雷达位置，更新雷达参数，添加音频文件

File: Nodes/sam_bot_description/src/description/simple_bot.urdf (robot description, URDF)
Before this commit: robot simple_bot, 2 links, 1 joints
Joints:
- joint lidar_joint: origin xyz=${-wheel_base/2} ${wheel_separation/2 - 0.09} ${-base_height/2 + wheel_radius + 0.19} rpy=0 0 0 -> xyz=-2.25 0 ${-base_height/2 + wheel_radius + 0.19} rpy=0 0 0

Commit message: 修复雷达位置错误，增碰撞预防器

File: Nodes/sam_bot_description/src/description/simple_bot.urdf (robot description, URDF)
Before this commit: robot simple_bot, 2 links, 1 joints
Joints:
- joint lidar_joint: origin xyz=-2.25 0 ${-base_height/2 + wheel_radius + 0.19} rpy=0 0 0 -> xyz=-0.0225 0 ${-base_height/2 + wheel_radius + 0.19} rpy=0 0 0
